File: board/sign/schematic.brd (EAGLE design)
At the start: 97.8 x 65.7 mm, 37 parts, among them IC1 STM32F207ZGT, IC3 LM3940, J1 DCJ0202, X2 22-23-2041

Commit message: Board REV A done
Parts:
- C24: device rcl:PANASONIC_A -> rcl:E2-5
- JP2: device con-lstb:MA04-1 -> con-lstb:MA05-1
- moved C23 3.86 mm to (14.0, 21.0)
- moved C24 3.18 mm to (15.2, 27.3)
- moved R3 2.54 mm to (90.2, 30.5)
- moved R4 2.54 mm to (92.7, 29.2)
- moved R2 1.27 mm to (95.2, 27.9)
Connections:
- net DEBUG_TX: now also JP2.5
Routing:
- net RESET: track 0.00 -> 104.9 mm, vias 0 -> 2
- net RX: track 0.00 -> 65.6 mm
- net +3V3: track 12.6 -> 71.1 mm, vias 0 -> 1
- net B: track 0.00 -> 48.5 mm
- net R0: track 0.00 -> 47.6 mm
- net A: track 0.00 -> 47.0 mm
- net GND: track 11.8 -> 58.6 mm, vias 0 -> 4
- net R1: track 0.00 -> 46.0 mm, vias 0 -> 1
- net B0: track 0.00 -> 45.2 mm
- net DCLK: track 0.00 -> 44.0 mm, vias 0 -> 1
- net C: track 0.00 -> 43.5 mm
- net B1: track 0.00 -> 43.4 mm, vias 0 -> 1
- net G0: track 0.00 -> 43.0 mm
- net DEBUG_TX: track 0.00 -> 37.4 mm
- net G1: track 0.00 -> 36.7 mm, vias 0 -> 1
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Other:
- board text added: "DISP DATA"
- board text added: "DISP POWER"
- board text added: "ESP DEBUG"
- board text added: "STM DEBUG"

Commit message: Please merge this outline change?
Other:
- board size 97.8 x 65.7 mm -> 97.8 x 65.8 mm
Changed lines of the file:
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@@
 <board>
 <plain>
-<wire x1="0" y1="0" x2="97.77" y2="0" width="0" layer="20"/>
-<wire x1="97.77" y1="0" x2="97.77" y2="58.09" width="0" layer="20"/>
-<wire x1="97.77" y1="58.09" x2="0" y2="65.71" width="0" layer="20"/>
-<wire x1="0" y1="65.71" x2="0" y2="0" width="0" layer="20"/>
 <text x="2.54" y="59.69" size="1.3208" layer="21">RESET</text>
 <text x="34.29" y="2.032" size="1.3208" layer="21">R0</text>
@@
 <text x="26.67" y="10.16" size="1.778" layer="21">GND</text>
 <text x="76.2" y="7.62" size="1.778" layer="21">SD</text>
-<text x="20.447" y="55.626" size="1.905" layer="21">MSign
+<text x="19.304" y="58.166" size="1.905" layer="21">MSign
 Rev A</text>
 <hole x="43.815" y="58.42" drill="3.2"/>
 <hole x="20.955" y="16.51" drill="3.2"/>
-<hole x="90.805" y="8.89" drill="3.2"/>
-<wire x1="19.05" y1="60.96" x2="29.21" y2="60.96" width="0.1524" layer="21"/>
-<wire x1="29.21" y1="60.96" x2="29.21" y2="54.61" width="0.1524" layer="21"/>
-<wire x1="29.21" y1="54.61" x2="19.05" y2="54.61" width="0.1524" layer="21"/>
-<wire x1="19.05" y1="54.61" x2="19.05" y2="60.96" width="0.1524" layer="21"/>
+<hole x="90.424" y="16.129" drill="3.2"/>
+<wire x1="17.907" y1="63.5" x2="28.067" y2="63.5" width="0.1524" layer="21"/>
+<wire x1="28.067" y1="63.5" x2="28.067" y2="57.15" width="0.1524" layer="21"/>
+<wire x1="28.067" y1="57.15" x2="17.907" y2="57.15" width="0.1524" layer="21"/>
+<wire x1="17.907" y1="57.15" x2="17.907" y2="63.5" width="0.1524" layer="21"/>
 <text x="18.415" y="1.27" size="1.27" layer="21">DISP POWER</text>
 <text x="37.465" y="1.905" size="1.27" layer="21">DISP DATA</text>
@@
 <dimension x1="0" y1="0" x2="0" y2="65.786" x3="-7.62" y3="32.893" textsize="1.27" layer="20"/>
 <dimension x1="97.79" y1="0" x2="0" y2="0" x3="48.895" y3="-7.62" textsize="1.27" layer="20"/>
+<wire x1="0" y1="0" x2="97.79" y2="0" width="0.0762" layer="20"/>
+<wire x1="97.79" y1="0" x2="97.79" y2="58.42" width="0.0762" layer="20"/>
+<wire x1="97.79" y1="58.42" x2="93.472" y2="62.738" width="0.0762" layer="20"/>
+<wire x1="93.472" y1="62.738" x2="31.242" y2="62.738" width="0.0762" layer="20"/>
+<wire x1="31.242" y1="62.738" x2="28.194" y2="65.786" width="0.0762" layer="20"/>
+<wire x1="28.194" y1="65.786" x2="0" y2="65.786" width="0.0762" layer="20"/>
+<wire x1="0" y1="65.786" x2="0" y2="0" width="0.0762" layer="20"/>
 </plain>
 <attributes>
@@
 <contactref element="IC3" pad="2"/>
 <polygon width="0.1524" layer="1" isolate="0.3302">
-<vertex x="0" y="66.04"/>
-<vertex x="97.79" y="58.42"/>
+<vertex x="0" y="69.723"/>
+<vertex x="97.79" y="62.103"/>
 <vertex x="97.79" y="0"/>
 <vertex x="0" y="0"/>
@@
 <wire x1="57.672959375" y1="28.033090625" x2="57.14625" y2="28.5598" width="0.3048" layer="1"/>
 <via x="41.91" y="17.78" extent="1-16" drill="0.35"/>
-<via x="43.815" y="21.59" extent="1-16" drill="0.35"/>
-<wire x1="39.37" y1="21.59" x2="41.91" y2="19.05" width="0.3048" layer="1"/>
-<wire x1="41.91" y1="19.05" x2="41.91" y2="17.78" width="0.3048" layer="1"/>
-<wire x1="43.815" y1="21.59" x2="42.911925" y2="22.493075" width="0.3048" layer="1"/>
-<wire x1="42.911925" y1="22.493075" x2="42.911925" y2="22.94045625" width="0.3048" layer="1"/>
-<wire x1="41.91" y1="17.78" x2="41.91" y2="19.685" width="0.3048" layer="16"/>
-<wire x1="41.91" y1="19.685" x2="43.815" y2="21.59" width="0.3048" layer="16"/>
+<via x="42.926" y="21.209" extent="1-16" drill="0.35"/>
+<wire x1="40.767" y1="17.78" x2="39.37" y2="19.177" width="0.3048" layer="1"/>
+<wire x1="39.37" y1="21.59" x2="39.37" y2="19.177" width="0.3048" layer="1"/>
+<wire x1="40.767" y1="17.78" x2="41.91" y2="17.78" width="0.3048" layer="1"/>
+<wire x1="42.926" y1="21.209" x2="42.911925" y2="21.223075" width="0.3048" layer="1"/>
+<wire x1="42.911925" y1="21.223075" x2="42.911925" y2="22.94045625" width="0.3048" layer="1"/>
+<wire x1="41.91" y1="17.78" x2="41.91" y2="20.193" width="0.3048" layer="16"/>
+<wire x1="41.91" y1="20.193" x2="42.926" y2="21.209" width="0.3048" layer="16"/>
 <via x="70.485" y="20.32" extent="1-16" drill="0.35"/>
 <via x="75.565" y="22.86" extent="1-16" drill="0.35"/>
@@
 <contactref element="IC1" pad="144"/>
 <polygon width="0.1524" layer="16" isolate="0.3048">
-<vertex x="0" y="65.786"/>
-<vertex x="97.79" y="58.166"/>
+<vertex x="0" y="69.723"/>
+<vertex x="97.79" y="62.103"/>
 <vertex x="97.79" y="0"/>
 <vertex x="0" y="0"/>
@@
 <wire x1="77.47" y1="20.32" x2="76.57" y2="19.42" width="0.3048" layer="1"/>
 <wire x1="76.57" y1="19.42" x2="76.57" y2="16.59" width="0.3048" layer="1"/>
-<wire x1="53.2863875" y1="20.614996875" x2="53.2863875" y2="24.0763875" width="0.3048" layer="1"/>
-<wire x1="53.2863875" y1="24.0763875" x2="53.34" y2="24.13" width="0.3048" layer="1"/>
+<wire x1="53.34" y1="24.13" x2="53.34" y2="20.668609375" width="0.3048" layer="1"/>
+<wire x1="53.2863875" y1="20.614996875" x2="53.34" y2="20.668609375" width="0.3048" layer="1"/>
 <wire x1="52.9902" y1="25.40375" x2="52.9902" y2="26.1848" width="0.3048" layer="1"/>
 <wire x1="52.9902" y1="26.1848" x2="52.97" y2="26.205" width="0.3048" layer="1"/>
@@
 <wire x1="53.34" y1="25.05395" x2="52.9902" y2="25.40375" width="0.3048" layer="1"/>
 <wire x1="52.97" y1="26.205" x2="52.47" y2="26.205" width="0.3048" layer="1"/>
-<wire x1="48.152771875" y1="22.806365625" x2="50.57160625" y2="25.2252" width="0.3048" layer="1"/>
-<wire x1="50.57160625" y1="25.2252" x2="51.27125" y2="25.2252" width="0.3048" layer="1"/>
-<wire x1="51.27125" y1="25.2252" x2="51.47" y2="25.42395" width="0.3048" layer="1"/>
+<wire x1="48.152771875" y1="22.806365625" x2="49.80960625" y2="24.4632" width="0.3048" layer="1"/>
+<wire x1="49.80960625" y1="24.4632" x2="50.50925" y2="24.4632" width="0.3048" layer="1"/>
+<wire x1="50.50925" y1="24.4632" x2="51.47" y2="25.42395" width="0.3048" layer="1"/>
 <wire x1="51.47" y1="25.42395" x2="51.47" y2="26.205" width="0.3048" layer="1"/>
 <wire x1="44.9902" y1="25.40375" x2="44.9902" y2="26.1848" width="0.3048" layer="1"/>
@@
 <wire x1="95.25" y1="31.75" x2="88.4" y2="31.75" width="0.1524" layer="1"/>
 <wire x1="87.32" y1="30.67" x2="88.4" y2="31.75" width="0.1524" layer="1"/>
-<wire x1="86.0914" y1="35.3646875" x2="86.2253125" y2="35.4986" width="0.1524" layer="1"/>
 <wire x1="87.32" y1="30.67" x2="87.32" y2="30.7467125" width="0.1524" layer="1"/>
-<wire x1="86.2253125" y1="35.4986" x2="86.2986" y2="35.4986" width="0.1524" layer="1"/>
 <wire x1="87.32" y1="30.7467125" x2="86.0914" y2="31.9753125" width="0.1524" layer="1"/>
 <wire x1="86.0914" y1="31.9753125" x2="86.0914" y2="35.3646875" width="0.1524" layer="1"/>
-<wire x1="86.6414" y1="35.8414" x2="88.4146875" y2="35.8414" width="0.1524" layer="1"/>
+<wire x1="86.5681125" y1="35.8414" x2="88.4146875" y2="35.8414" width="0.1524" layer="1"/>
 <wire x1="88.4146875" y1="35.8414" x2="88.9" y2="36.3267125" width="0.1524" layer="1"/>
-<wire x1="86.2986" y1="35.4986" x2="86.6414" y2="35.8414" width="0.1524" layer="1"/>
+<wire x1="86.0914" y1="35.3646875" x2="86.5681125" y2="35.8414" width="0.1524" layer="1"/>
 <wire x1="78.62" y1="39.37" x2="74.4914" y2="43.4986" width="0.1524" layer="1"/>
 <wire x1="85.66565625" y1="39.37" x2="78.62" y2="39.37" width="0.1524" layer="1"/>
