File: board/sign/schematic.sch (EAGLE design)
At the start: 40 parts, among them IC1 STM32F207ZGT, IC3 LM3940, J1 DCJ0202, J3 DM3AT-SF-PEJM5, X2 22-23-2041

Commit message: Fix board FINAL
Connections:
- removed net N$4: C18.2, JP1.13
- net DCLK: now also C18.2, JP1.13; no longer C18.1
- net GND: now also C18.1
Other:
- moved on the sheet: C18
Changed lines of the file:
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@@
 <part name="J3" library="connector" deviceset="DM3AT-SF-PEJM5" device=""/>
 <part name="C18" library="rcl" library_urn="urn:adsk.eagle:library:334" deviceset="C-EU" device="050-024X044" package3d_urn="urn:adsk.eagle:package:23643/1" value="10pF"/>
+<part name="GND21" library="supply1" library_urn="urn:adsk.eagle:library:371" deviceset="GND" device=""/>
 </parts>
 <sheets>
@@
 <attribute name="VALUE" x="205.74" y="68.58" size="1.27" layer="96"/>
 </instance>
-<instance part="C18" gate="G$1" x="274.32" y="68.58" smashed="yes" rot="R90">
-<attribute name="NAME" x="273.939" y="70.104" size="1.778" layer="95" rot="R90"/>
-<attribute name="VALUE" x="279.019" y="70.104" size="1.778" layer="96" rot="R90"/>
+<instance part="C18" gate="G$1" x="274.32" y="63.5" smashed="yes" rot="R180">
+<attribute name="NAME" x="272.796" y="63.119" size="1.778" layer="95" rot="R180"/>
+<attribute name="VALUE" x="272.796" y="68.199" size="1.778" layer="96" rot="R180"/>
+</instance>
+<instance part="GND21" gate="1" x="274.32" y="58.42" smashed="yes">
+<attribute name="VALUE" x="271.78" y="55.88" size="1.778" layer="96"/>
 </instance>
 </instances>
@@
 </segment>
 <segment>
-<pinref part="C18" gate="G$1" pin="1"/>
-<wire x1="271.78" y1="68.58" x2="259.08" y2="68.58" width="0.1524" layer="91"/>
+<pinref part="JP1" gate="A" pin="13"/>
+<pinref part="C18" gate="G$1" pin="2"/>
+<wire x1="297.18" y1="68.58" x2="274.32" y2="68.58" width="0.1524" layer="91"/>
+<wire x1="274.32" y1="68.58" x2="259.08" y2="68.58" width="0.1524" layer="91"/>
+<junction x="274.32" y="68.58"/>
 <label x="259.08" y="68.58" size="1.778" layer="95"/>
 </segment>
@@
 <pinref part="GND4" gate="1" pin="GND"/>
 </segment>
+<segment>
+<pinref part="C18" gate="G$1" pin="1"/>
+<pinref part="GND21" gate="1" pin="GND"/>
+</segment>
 </net>
 <net name="+3V3" class="0">
@@
 </segment>
 </net>
-<net name="N$4" class="0">
-<segment>
-<pinref part="JP1" gate="A" pin="13"/>
-<pinref part="C18" gate="G$1" pin="2"/>
-<wire x1="297.18" y1="68.58" x2="279.4" y2="68.58" width="0.1524" layer="91"/>
-</segment>
-</net>

Commit message: Actually the final board I promise
Parts:
- removed X2: 22-23-2041, con-molex:22-23-2041
- added C25: 100nF, rcl:C-EU025-025X050
- added J2: (no value), SparkFun-Connectors:CONN_025MM
Connections:
- net +3V3: now also C25.1
- net +5V: now also J2.1; no longer X2-1.S, X2-2.S
- net GND: now also C25.2, J2.2; no longer X2-3.S, X2-4.S
Changed lines of the file:
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@@
 <layer number="56" name="wert" color="7" fill="1" visible="no" active="no"/>
 <layer number="57" name="tCAD" color="7" fill="1" visible="no" active="no"/>
+<layer number="59" name="tCarbon" color="7" fill="1" visible="no" active="no"/>
+<layer number="60" name="bCarbon" color="7" fill="1" visible="no" active="no"/>
 <layer number="88" name="SimResults" color="9" fill="1" visible="yes" active="yes"/>
 <layer number="89" name="SimProbes" color="9" fill="1" visible="yes" active="yes"/>
@@
 <layer number="112" name="tSilk" color="7" fill="1" visible="yes" active="yes"/>
 <layer number="113" name="IDFDebug" color="7" fill="1" visible="yes" active="yes"/>
+<layer number="114" name="Badge_Outline" color="7" fill="1" visible="no" active="no"/>
+<layer number="115" name="ReferenceISLANDS" color="7" fill="1" visible="no" active="no"/>
 <layer number="116" name="Patch_BOT" color="9" fill="4" visible="yes" active="yes"/>
+<layer number="118" name="Rect_Pads" color="7" fill="1" visible="no" active="no"/>
 <layer number="121" name="_tsilk" color="7" fill="1" visible="yes" active="yes"/>
 <layer number="122" name="_bsilk" color="7" fill="1" visible="yes" active="yes"/>
@@
 <layer number="127" name="_tValues" color="7" fill="1" visible="yes" active="yes"/>
 <layer number="128" name="_bValues" color="7" fill="1" visible="yes" active="yes"/>
+<layer number="129" name="Mask" color="7" fill="1" visible="no" active="no"/>
 <layer number="131" name="tAdjust" color="7" fill="1" visible="no" active="yes"/>
 <layer number="132" name="bAdjust" color="7" fill="1" visible="no" active="yes"/>
@@
 <layer number="223" name="223bmp" color="24" fill="1" visible="no" active="no"/>
 <layer number="224" name="224bmp" color="25" fill="1" visible="no" active="no"/>
+<layer number="225" name="225bmp" color="7" fill="1" visible="no" active="no"/>
+<layer number="226" name="226bmp" color="7" fill="1" visible="no" active="no"/>
+<layer number="227" name="227bmp" color="7" fill="1" visible="no" active="no"/>
+<layer number="228" name="228bmp" color="7" fill="1" visible="no" active="no"/>
+<layer number="229" name="229bmp" color="7" fill="1" visible="no" active="no"/>
+<layer number="230" name="230bmp" color="7" fill="1" visible="no" active="no"/>
+<layer number="231" name="231bmp" color="7" fill="1" visible="no" active="no"/>
+<layer number="232" name="Eagle3D_PG2" color="7" fill="1" visible="no" active="no"/>
+<layer number="233" name="Eagle3D_PG3" color="7" fill="1" visible="no" active="no"/>
 <layer number="248" name="Housing" color="7" fill="1" visible="yes" active="yes"/>
 <layer number="249" name="Edge" color="7" fill="1" visible="yes" active="yes"/>
@@
 <layer number="251" name="SMDround" color="7" fill="1" visible="no" active="no"/>
 <layer number="254" name="cooling" color="7" fill="1" visible="yes" active="yes"/>
+<layer number="255" name="routoute" color="7" fill="1" visible="no" active="no"/>
 </layers>
 <schematic xreflabel="%F%N/%S.%C%R" xrefpart="/%S.%C%R">
@@
 <part name="C21" library="rcl" library_urn="urn:adsk.eagle:library:334" deviceset="C-EU" device="025-025X050" package3d_urn="urn:adsk.eagle:package:23629/2" value="100nF"/>
 <part name="GND13" library="supply1" library_urn="urn:adsk.eagle:library:371" deviceset="GND" device=""/>
-<part name="X2" library="con-molex" library_urn="urn:adsk.eagle:library:165" deviceset="22-23-2041" device=""/>
 <part name="P+1" library="supply1" library_urn="urn:adsk.eagle:library:371" deviceset="+5V" device=""/>
 <part name="GND14" library="supply1" library_urn="urn:adsk.eagle:library:371" deviceset="GND" device=""/>
@@
 <part name="C18" library="rcl" library_urn="urn:adsk.eagle:library:334" deviceset="C-EU" device="050-024X044" package3d_urn="urn:adsk.eagle:package:23643/1" value="10pF"/>
 <part name="GND21" library="supply1" library_urn="urn:adsk.eagle:library:371" deviceset="GND" device=""/>
+<part name="J2" library="SparkFun-Connectors" deviceset="CONN_02" device="5MM"/>
+<part name="C25" library="rcl" library_urn="urn:adsk.eagle:library:334" deviceset="C-EU" device="025-025X050" package3d_urn="urn:adsk.eagle:package:23629/2" value="100nF"/>
+<part name="GND22" library="supply1" library_urn="urn:adsk.eagle:library:371" deviceset="GND" device=""/>
 </parts>
 <sheets>
@@
 <attribute name="NAME" x="40.64" y="50.8" size="1.27" layer="94"/>
 </instance>
-<instance part="+3V3" gate="G$1" x="10.16" y="27.94" smashed="yes" rot="R90">
-<attribute name="VALUE" x="15.24" y="25.4" size="1.778" layer="96" rot="R180"/>
+<instance part="+3V3" gate="G$1" x="-2.54" y="27.94" smashed="yes" rot="R90">
+<attribute name="VALUE" x="2.54" y="25.4" size="1.778" layer="96" rot="R180"/>
 </instance>
 <instance part="GND8" gate="1" x="73.66" y="27.94" smashed="yes" rot="R90">
@@
 <attribute name="VALUE" x="238.76" y="119.38" size="1.778" layer="96" rot="R180"/>
 </instance>
-<instance part="X2" gate="-1" x="162.56" y="127" smashed="yes">
-<attribute name="NAME" x="165.1" y="126.238" size="1.524" layer="95"/>
-<attribute name="VALUE" x="161.798" y="128.397" size="1.778" layer="96"/>
-</instance>
-<instance part="X2" gate="-2" x="162.56" y="124.46" smashed="yes">
-<attribute name="NAME" x="165.1" y="123.698" size="1.524" layer="95"/>
-</instance>
-<instance part="X2" gate="-3" x="162.56" y="121.92" smashed="yes">
-<attribute name="NAME" x="165.1" y="121.158" size="1.524" layer="95"/>
-</instance>
-<instance part="X2" gate="-4" x="162.56" y="119.38" smashed="yes">
-<attribute name="NAME" x="165.1" y="118.618" size="1.524" layer="95"/>
-</instance>
 <instance part="P+1" gate="1" x="152.4" y="137.16" smashed="yes">
 <attribute name="VALUE" x="149.86" y="132.08" size="1.778" layer="96" rot="R90"/>
@@
 <instance part="GND21" gate="1" x="274.32" y="58.42" smashed="yes">
 <attribute name="VALUE" x="271.78" y="55.88" size="1.778" layer="96"/>
+</instance>
+<instance part="J2" gate="G$1" x="167.64" y="124.46" smashed="yes" rot="R180">
+<attribute name="VALUE" x="170.18" y="129.286" size="1.778" layer="96" font="vector" rot="R180"/>
+<attribute name="NAME" x="170.18" y="118.872" size="1.778" layer="95" font="vector" rot="R180"/>
+</instance>
+<instance part="C25" gate="G$1" x="7.62" y="25.4" smashed="yes">
+<attribute name="NAME" x="9.144" y="25.781" size="1.778" layer="95"/>
+<attribute name="VALUE" x="9.144" y="20.701" size="1.778" layer="96"/>
+</instance>
+<instance part="GND22" gate="1" x="7.62" y="17.78" smashed="yes">
+<attribute name="VALUE" x="5.08" y="15.24" size="1.778" layer="96"/>
 </instance>
 </instances>
@@
 <segment>
 <pinref part="GND14" gate="1" pin="GND"/>
-<wire x1="152.4" y1="114.3" x2="152.4" y2="119.38" width="0.1524" layer="91"/>
-<pinref part="X2" gate="-4" pin="S"/>
-<wire x1="152.4" y1="119.38" x2="160.02" y2="119.38" width="0.1524" layer="91"/>
-<pinref part="X2" gate="-3" pin="S"/>
+<wire x1="152.4" y1="114.3" x2="152.4" y2="121.92" width="0.1524" layer="91"/>
 <wire x1="160.02" y1="121.92" x2="152.4" y2="121.92" width="0.1524" layer="91"/>
-<wire x1="152.4" y1="121.92" x2="152.4" y2="119.38" width="0.1524" layer="91"/>
-<junction x="152.4" y="119.38"/>
+<pinref part="J2" gate="G$1" pin="2"/>
 </segment>
 <segment>
@@
 <pinref part="C18" gate="G$1" pin="1"/>
 <pinref part="GND21" gate="1" pin="GND"/>
+</segment>
+<segment>
+<pinref part="C25" gate="G$1" pin="2"/>
+<pinref part="GND22" gate="1" pin="GND"/>
 </segment>
 </net>
@@
 <pinref part="+3V3" gate="G$1" pin="+3V3"/>
 <pinref part="IC2" gate="G$1" pin="VCC"/>
-<wire x1="12.7" y1="27.94" x2="20.32" y2="27.94" width="0.1524" layer="91"/>
+<wire x1="0" y1="27.94" x2="7.62" y2="27.94" width="0.1524" layer="91"/>
 <pinref part="C19" gate="G$1" pin="+"/>
+<wire x1="7.62" y1="27.94" x2="20.32" y2="27.94" width="0.1524" layer="91"/>
 <wire x1="20.32" y1="27.94" x2="27.94" y2="27.94" width="0.1524" layer="91"/>
 <junction x="20.32" y="27.94"/>
+<pinref part="C25" gate="G$1" pin="1"/>
+<junction x="7.62" y="27.94"/>
 </segment>
 <segment>
@@
 <net name="+5V" class="0">
 <segment>
-<pinref part="X2" gate="-1" pin="S"/>
 <pinref part="P+1" gate="1" pin="+5V"/>
-<wire x1="160.02" y1="127" x2="152.4" y2="127" width="0.1524" layer="91"/>
-<wire x1="152.4" y1="127" x2="152.4" y2="134.62" width="0.1524" layer="91"/>
-<wire x1="152.4" y1="127" x2="152.4" y2="124.46" width="0.1524" layer="91"/>
-<junction x="152.4" y="127"/>
-<pinref part="X2" gate="-2" pin="S"/>
+<wire x1="152.4" y1="124.46" x2="152.4" y2="134.62" width="0.1524" layer="91"/>
 <wire x1="152.4" y1="124.46" x2="160.02" y2="124.46" width="0.1524" layer="91"/>
-</segment>
-<segment>
+<pinref part="J2" gate="G$1" pin="1"/>
+</segment>
+<segment>
