File: board/schematic.brd (EAGLE design)
At the start: 97.8 x 65.8 mm, 41 parts, among them IC1 STM32F207ZGT, IC3 LM3940, J1 DCJ0202, J3 DM3AT-SF-PEJM5

Commit message: Board w/ more measures; final version is still on my computer
Parts:
- removed JP3: (no value), con-lstb:MA06-1
- added J4: (no value), pinhead:2X08
- JP1: device pinhead:2X08 -> pinhead:1X05
- JP2: device con-lstb:MA05-1 -> con-lstb:MA06-1
- moved JP1 61.0 mm to (80.0, 55.9)
- moved JP2 59.3 mm to (21.6, 45.7), turned to 90 degrees
Connections:
- net +3V3: now also JP1.1; no longer JP3.1
- net A: now also J4.9; no longer JP1.9
- net B: now also J4.10; no longer JP1.10
- net B0: now also J4.3; no longer JP1.3
- net B1: now also J4.7; no longer JP1.7
- net C: now also J4.11; no longer JP1.11
- net D: now also J4.12; no longer JP1.12
- net DCLK: now also J4.13; no longer JP1.13
- net DEBUG_TX: now also JP1.5; no longer JP2.5
- net ESP_PROG_RX: now also JP1.3; no longer JP2.3
- net ESP_PROG_TX: now also JP1.2; no longer JP2.2
- net G0: now also J4.2; no longer JP1.2
- net G1: now also J4.6; no longer JP1.6
- net GND: now also J4.16, J4.4, J4.8, JP2.3; no longer JP1.16, JP1.8, JP2.4, JP3.3
- net LAT: now also J4.14; no longer JP1.14
- net OE: now also J4.15; no longer JP1.15
- net R0: now also J4.1; no longer JP1.1
- net R1: now also J4.5; no longer JP1.5
- net RESET: now also JP2.5; no longer JP3.5
- net SWCLK: now also JP2.2; no longer JP3.2
- net SWDIO: now also JP2.4; no longer JP3.4
Other:
- board text added: "This page intentionally left blank"
Changed lines of the file:
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@@
 <wire x1="65.024" y1="18.034" x2="53.467" y2="18.034" width="0.1524" layer="22"/>
 <wire x1="53.467" y1="18.034" x2="53.467" y2="11.684" width="0.1524" layer="22"/>
+<dimension x1="97.79" y1="0" x2="97.79" y2="58.42" x3="108.204" y3="29.21" textsize="1.778" layer="47"/>
+<text x="84.455" y="46.101" size="0.8128" layer="22" rot="MR0">This page intentionally
+left blank</text>
 </plain>
 <attributes>
@@
 <attribute name="VALUE" x="2.54" y="1.27" size="1.27" layer="27" rot="R90"/>
 </element>
-<element name="JP1" library="pinhead" library_urn="urn:adsk.eagle:library:325" package="2X08" package3d_urn="urn:adsk.eagle:package:22481/2" value="" x="44.45" y="6.35" smashed="yes">
+<element name="J4" library="pinhead" library_urn="urn:adsk.eagle:library:325" package="2X08" package3d_urn="urn:adsk.eagle:package:22481/2" value="" x="44.45" y="6.35" smashed="yes">
 <attribute name="NAME" x="34.29" y="9.525" size="1.27" layer="25" ratio="10"/>
 <attribute name="VALUE" x="34.29" y="1.905" size="1.27" layer="27"/>
 </element>
-<element name="JP2" library="con-lstb" library_urn="urn:adsk.eagle:library:162" package="MA05-1" package3d_urn="urn:adsk.eagle:package:8332/1" value="" x="80.01" y="55.88" smashed="yes">
-<attribute name="MF" value="" x="125.73" y="-17.78" size="1.778" layer="27" display="off"/>
-<attribute name="MPN" value="" x="125.73" y="-17.78" size="1.778" layer="27" display="off"/>
+<element name="JP1" library="pinhead" library_urn="urn:adsk.eagle:library:325" package="1X05" package3d_urn="urn:adsk.eagle:package:22469/2" value="" x="80.01" y="55.88" smashed="yes">
 <attribute name="NAME" x="74.93" y="57.531" size="1.27" layer="25" ratio="10"/>
-<attribute name="OC_FARNELL" value="unknown" x="125.73" y="-17.78" size="1.778" layer="27" display="off"/>
-<attribute name="OC_NEWARK" value="unknown" x="125.73" y="-17.78" size="1.778" layer="27" display="off"/>
 <attribute name="VALUE" x="80.645" y="57.531" size="1.27" layer="27" ratio="10"/>
 </element>
-<element name="JP3" library="con-lstb" library_urn="urn:adsk.eagle:library:162" package="MA06-1" package3d_urn="urn:adsk.eagle:package:8340/1" value="" x="21.59" y="45.72" smashed="yes" rot="R90">
+<element name="JP2" library="con-lstb" library_urn="urn:adsk.eagle:library:162" package="MA06-1" package3d_urn="urn:adsk.eagle:package:8340/1" value="" x="21.59" y="45.72" smashed="yes" rot="R90">
 <attribute name="MF" value="" x="73.66" y="99.06" size="1.778" layer="27" rot="R90" display="off"/>
 <attribute name="MPN" value="" x="73.66" y="99.06" size="1.778" layer="27" rot="R90" display="off"/>
@@
 <signal name="R0">
 <contactref element="IC1" pad="114"/>
-<contactref element="JP1" pad="1"/>
+<contactref element="J4" pad="1"/>
 <wire x1="35.095" y1="43.08" x2="30.38" y2="43.08" width="0.1524" layer="1"/>
 <wire x1="28.067" y1="40.767" x2="28.067" y2="13.462" width="0.1524" layer="1"/>
@@
 <signal name="G0">
 <contactref element="IC1" pad="115"/>
-<contactref element="JP1" pad="2"/>
+<contactref element="J4" pad="2"/>
 <wire x1="35.095" y1="42.58" x2="30.642" y2="42.58" width="0.1524" layer="1"/>
 <wire x1="30.642" y1="42.58" x2="28.448" y2="40.386" width="0.1524" layer="1"/>
@@
 <signal name="B0">
 <contactref element="IC1" pad="116"/>
-<contactref element="JP1" pad="3"/>
+<contactref element="J4" pad="3"/>
 <wire x1="35.095" y1="42.08" x2="30.904" y2="42.08" width="0.1524" layer="1"/>
 <wire x1="30.904" y1="42.08" x2="28.956" y2="40.132" width="0.1524" layer="1"/>
@@
 <signal name="R1">
 <contactref element="IC1" pad="117"/>
-<contactref element="JP1" pad="5"/>
+<contactref element="J4" pad="5"/>
 <via x="39.37" y="36.83" extent="1-16" drill="0.35"/>
 <wire x1="35.095" y1="41.58" x2="35.1914" y2="41.4836" width="0.1524" layer="1"/>
@@
 <signal name="G1">
 <contactref element="IC1" pad="118"/>
-<contactref element="JP1" pad="6"/>
+<contactref element="J4" pad="6"/>
 <via x="40.64" y="35.56" extent="1-16" drill="0.35"/>
 <wire x1="35.095" y1="41.08" x2="35.1914" y2="40.9836" width="0.1524" layer="1"/>
@@
 <signal name="B1">
 <contactref element="IC1" pad="119"/>
-<contactref element="JP1" pad="7"/>
+<contactref element="J4" pad="7"/>
 <via x="33.274" y="41.402" extent="1-16" drill="0.35"/>
 <wire x1="35.095" y1="40.58" x2="34.35276875" y2="40.58" width="0.1524" layer="1"/>
@@
 <wire x1="50.8" y1="31.369" x2="50.8" y2="27.94" width="0.1524" layer="1"/>
 <wire x1="40.0784875" y1="34.7698" x2="47.3992" y2="34.7698" width="0.1524" layer="1"/>
-<contactref element="JP1" pad="13"/>
+<contactref element="J4" pad="13"/>
 <contactref element="C18" pad="2"/>
 <wire x1="56.769" y1="7.62" x2="56.769" y2="5.715" width="0.1524" layer="16"/>
@@
 <signal name="A">
 <contactref element="IC1" pad="46"/>
-<contactref element="JP1" pad="9"/>
+<contactref element="J4" pad="9"/>
 <wire x1="55.5753125" y1="32.4836" x2="55.4414" y2="32.3496875" width="0.1524" layer="1"/>
 <wire x1="55.4414" y1="32.3496875" x2="55.4414" y2="27.8103125" width="0.1524" layer="1"/>
@@
 <signal name="B">
 <contactref element="IC1" pad="47"/>
-<contactref element="JP1" pad="10"/>
+<contactref element="J4" pad="10"/>
 <wire x1="55.1366" y1="27.68405625" x2="55.49025625" y2="27.3304" width="0.1524" layer="1"/>
 <wire x1="55.49025625" y1="27.3304" x2="56.97471875" y2="27.3304" width="0.1524" layer="1"/>
@@
 <signal name="C">
 <contactref element="IC1" pad="48"/>
-<contactref element="JP1" pad="11"/>
+<contactref element="J4" pad="11"/>
 <wire x1="56.345" y1="33.58" x2="56.2486" y2="33.4836" width="0.1524" layer="1"/>
 <wire x1="56.2486" y1="33.4836" x2="55.5753125" y2="33.4836" width="0.1524" layer="1"/>
@@
 <signal name="D">
 <contactref element="IC1" pad="133"/>
-<contactref element="JP1" pad="12"/>
+<contactref element="J4" pad="12"/>
 <via x="45.72" y="29.21" extent="1-16" drill="0.35"/>
 <wire x1="45.72" y1="29.21" x2="40.1382875" y2="29.21" width="0.1524" layer="1"/>
@@
 <signal name="LAT">
 <contactref element="IC1" pad="135"/>
-<contactref element="JP1" pad="14"/>
+<contactref element="J4" pad="14"/>
 <wire x1="35.095" y1="32.58" x2="35.1914" y2="32.4836" width="0.1524" layer="1"/>
 <wire x1="35.1914" y1="32.4836" x2="35.8646875" y2="32.4836" width="0.1524" layer="1"/>
@@
 <signal name="OE">
 <contactref element="IC1" pad="136"/>
-<contactref element="JP1" pad="15"/>
+<contactref element="J4" pad="15"/>
 <wire x1="35.095" y1="32.08" x2="35.1914" y2="31.9836" width="0.1524" layer="1"/>
 <wire x1="35.1914" y1="31.9836" x2="35.8646875" y2="31.9836" width="0.1524" layer="1"/>
@@
 <contactref element="S1" pad="3"/>
 <contactref element="C22" pad="2"/>
-<contactref element="JP1" pad="16"/>
-<contactref element="JP1" pad="8"/>
+<contactref element="J4" pad="16"/>
+<contactref element="J4" pad="8"/>
+<contactref element="J4" pad="4"/>
 <contactref element="JP1" pad="4"/>
-<contactref element="JP2" pad="4"/>
-<contactref element="JP3" pad="3"/>
+<contactref element="JP2" pad="3"/>
 <contactref element="C23" pad="2"/>
 <contactref element="C24" pad="-"/>
@@
 <contactref element="R3" pad="1"/>
 <contactref element="R4" pad="1"/>
+<contactref element="JP1" pad="1"/>
 <contactref element="JP2" pad="1"/>
-<contactref element="JP3" pad="1"/>
 <contactref element="IC3" pad="3"/>
 <contactref element="C24" pad="+"/>
@@
 <contactref element="R1" pad="1"/>
 <contactref element="C22" pad="1"/>
-<contactref element="JP3" pad="5"/>
+<contactref element="JP2" pad="5"/>
 <via x="48.26" y="29.21" extent="1-16" drill="0.35"/>
 <wire x1="6.35" y1="48.26" x2="6.35" y2="53.34" width="0.1524" layer="1"/>
@@
 <wire x1="87.32" y1="32.67" x2="87.67" y2="33.02" width="0.1524" layer="1"/>
 <wire x1="87.67" y1="33.02" x2="92.71" y2="33.02" width="0.1524" layer="1"/>
-<contactref element="JP2" pad="5"/>
+<contactref element="JP1" pad="5"/>
 <wire x1="92.71" y1="33.02" x2="92.71" y2="48.26" width="0.1524" layer="16"/>
 <wire x1="92.71" y1="48.26" x2="85.09" y2="55.88" width="0.1524" layer="16"/>
@@
 <signal name="ESP_PROG_TX">
 <contactref element="IC2" pad="16"/>
-<contactref element="JP2" pad="2"/>
+<contactref element="JP1" pad="2"/>
 <wire x1="87.32" y1="42.67" x2="89.025" y2="42.67" width="0.1524" layer="1"/>
 <wire x1="89.025" y1="42.67" x2="90.17" y2="43.815" width="0.1524" layer="1"/>
@@
 <signal name="ESP_PROG_RX">
 <contactref element="IC2" pad="15"/>
-<contactref element="JP2" pad="3"/>
+<contactref element="JP1" pad="3"/>
 <wire x1="87.32" y1="40.67" x2="91.47" y2="40.67" width="0.1524" layer="1"/>
 <wire x1="92.71" y1="50.8" x2="92.71" y2="41.91" width="0.1524" layer="1"/>
@@
 </signal>
 <signal name="SWDIO">
-<contactref element="JP3" pad="4"/>
+<contactref element="JP2" pad="4"/>
 <contactref element="IC1" pad="105"/>
 <wire x1="38.4498" y1="46.65375" x2="38.27125" y2="46.4752" width="0.1524" layer="1"/>
@@
 </signal>
 <signal name="SWCLK">
-<contactref element="JP3" pad="2"/>
+<contactref element="JP2" pad="2"/>
 <contactref element="IC1" pad="109"/>
 <wire x1="35.095" y1="45.58" x2="28.435" y2="45.58" width="0.1524" layer="1"/>
