File: board/contbrd.sch (EAGLE design)
At the start: 33 parts, among them IC1 74HCT244DW, IC3 LM3940, IC4 STM32F205RGT, IC5 74HCT244DW, J1 DCJ0202, J3 DM3AT-SF-PEJM5

Commit message: mb
Changed lines of the file:
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@@
 <?xml version="1.0" encoding="utf-8"?>
 <!DOCTYPE eagle SYSTEM "eagle.dtd">
-<eagle version="9.4.2">
+<eagle version="9.4.1">
 <drawing>
 <settings>
@@
 The STM and ESP</description>
 <plain>
-<wire x1="116.84" y1="5.08" x2="231.14" y2="5.08" width="0.254" layer="97"/>
+<wire x1="114.3" y1="5.08" x2="231.14" y2="5.08" width="0.254" layer="97"/>
 <wire x1="231.14" y1="5.08" x2="231.14" y2="114.3" width="0.254" layer="97"/>
-<wire x1="231.14" y1="114.3" x2="116.84" y2="114.3" width="0.254" layer="97"/>
-<wire x1="116.84" y1="114.3" x2="116.84" y2="5.08" width="0.254" layer="97"/>
+<wire x1="231.14" y1="114.3" x2="114.3" y2="114.3" width="0.254" layer="97"/>
+<wire x1="114.3" y1="114.3" x2="114.3" y2="5.08" width="0.254" layer="97"/>
 <wire x1="109.22" y1="5.08" x2="-7.62" y2="5.08" width="0.254" layer="97"/>
 <wire x1="-7.62" y1="5.08" x2="-7.62" y2="68.58" width="0.254" layer="97"/>

Commit message: board rev b
Parts:
- removed C19: 100uF, rcl:CPOL-USE2.5-6
- removed C21, C25: 100nF, rcl:C-EU025-025X050
- removed C22: 470pF, rcl:C-EU025-025X050
- removed C23: 0.47uF, rcl:C-EU050-024X044
- removed C24: 33uF, rcl:CPOL-USE2-5
- removed J3: DM3AT-SF-PEJM5, connector:DM3AT-SF-PEJM5
- added C10: 33uF, rcl:CPOL-USE2-5
- added C11, C12, C14: 100nF, rcl:C-EU025-025X050
- added C13: 470pF, rcl:C-EU025-025X050
- added C8: 0.47uF, rcl:C-EU050-024X044
- added JP4: (no value), pinhead:PINHD-1X9
- added JP5: (no value), pinhead:PINHD-1X6
- added R7: 12k, rcl:R-US_0204/7
- C2: value 1uF -> 100uF; device rcl:C-EU050-024X044 -> rcl:CPOL-USE2.5-6
- C3: value 100nF -> 1uF; device rcl:C-EU025-025X050 -> rcl:C-EU050-024X044
- C4: value 2.2uF -> 100nF; device rcl:CPOL-USE1.8-4 -> rcl:C-EU025-025X050
- C6: value 100nF -> 2.2uF; device rcl:C-EU025-025X050 -> rcl:CPOL-USE1.8-4
- IC1: value 74HCT244DW -> STM32F205RGT; device 74xx-eu:74HCT244DW -> micro-stm_v3:STM32F205RGT
- IC2: value (none) -> 74HCT244DW; device esp12e:ESP8266-12EESP12E -> 74xx-eu:74HCT244DW
- IC3: value LM3940 -> 74HCT244DW; device LM3940:LM3940 -> 74xx-eu:74HCT244DW
- IC4: value STM32F205RGT -> LM3940; device micro-stm_v3:STM32F205RGT -> LM3940:LM3940
- IC5: value 74HCT244DW -> (none); device 74xx-eu:74HCT244DW -> esp12e:ESP8266-12EESP12E
- JP1: value (none) -> DM3AT-SF-PEJM5; device pinhead:PINHD-1X5 -> connector:DM3AT-SF-PEJM5
- JP2: device con-lstb:MA06-1 -> pinhead:PINHD-1X5
- R4: value 12k -> 470
- R5: value 470 -> 12k
- renumbered C20 to C9, J5 to JP3
Connections:
- removed net N$4: C1.2, C2.2, C3.2, IC4MCU.VBAT, IC4MCU.VDDA
- new net ACTLED: IC1MCU.PA5, JP4.3
- new net MENBTN: IC1MCU.PA7, JP4.4
- new net NXTBTN: IC1MCU.PA10, JP4.6
- new net PRVBTN: IC1MCU.PA9, JP4.5
- new net PWRBTN: IC1MCU.PA0-WKUP, JP4.8, R7.1
- new net SELBTN: IC1MCU.PA8, JP4.7
- new net UPDLED: IC1MCU.PA6, JP4.2
- net +3V3: now also C1.1, C10.+, C11.1, C12.1, C14.1, C2.+, C3.2, C4.2, C7.2, IC1MCU.VBAT, IC1MCU.VDDA, IC1PWR.VDD@1, IC1PWR.VDD@2, IC1PWR.VDD@3, IC1PWR.VDD@4, IC4.OUT, IC5.CH_PD, IC5.VCC, JP1.VCC, JP4.1, JP5.1, R1.1, R2.1, R5.2; no longer C19.+, C21.1, C24.+, C25.1, C6.1, C7.1, IC2.CH_PD, IC2.VCC, IC3.OUT, IC4PWR.VDD@1, IC4PWR.VDD@2, IC4PWR.VDD@3, IC4PWR.VDD@4, J3.VCC, JP1.1, R1.2, R3.1, R4.1
- net +5V: now also C8.1, IC2P.VCC, IC3P.VCC, IC4.IN; no longer C23.1, IC1P.VCC, IC3.IN, IC5P.VCC
- net A: now also IC1MCU.PB0, IC3B.A1; no longer IC1B.A1, IC4MCU.PB0
- net A_H: now also IC3B.Y1; no longer IC1B.Y1
- net B: now also IC1MCU.PB1, IC2A.A3; no longer IC4MCU.PB1, IC5A.A3
- net B0: now also IC1MCU.PC2, IC3A.A2; no longer IC1A.A2, IC4MCU.PC2
- net B0_H: now also IC3A.Y2; no longer IC1A.Y2
- net B1: now also IC1MCU.PC5, IC3A.A4; no longer IC1A.A4, IC4MCU.PC5
- net B1_H: now also IC3A.Y4; no longer IC1A.Y4
- net B_H: now also IC2A.Y3; no longer IC5A.Y3
- net C: now also IC1MCU.PB2, IC3B.A2; no longer IC1B.A2, IC4MCU.PB2
- net C_H: now also IC3B.Y2; no longer IC1B.Y2
- net D: now also IC1MCU.PB3, IC2A.A4; no longer IC4MCU.PB3, IC5A.A4
- net DCLK: now also IC1MCU.PC6, IC3B.A3; no longer IC1B.A3, IC4MCU.PC6
- net DCLK_H: now also IC3B.Y3; no longer IC1B.Y3
- net DEBUG_TX: now also IC5.GPIO2, JP2.5, R2.2; no longer IC2.GPIO2, JP1.5, R4.2
- net D_H: now also IC2A.Y4; no longer IC5A.Y4
- net ESP_PROG_RX: now also IC5.RXD, JP2.3; no longer IC2.RXD, JP1.3
- net ESP_PROG_TX: now also IC5.TXD, JP2.2; no longer IC2.TXD, JP1.2
- net FLASH: now also IC5.GPIO0, R1.2, R4.2; no longer IC2.GPIO0, R3.2, R5.2
- net G0: now also IC1MCU.PC1, IC2A.A1; no longer IC4MCU.PC1, IC5A.A1
- net G0_H: now also IC2A.Y1; no longer IC5A.Y1
- net G1: now also IC1MCU.PC4, IC2A.A2; no longer IC4MCU.PC4, IC5A.A2
- net G1_H: now also IC2A.Y2; no longer IC5A.Y2
- net GND: now also C1.2, C10.-, C11.2, C12.2, C13.2, C14.2, C2.-, C4.1, C6.-, C7.1, C8.2, IC1MCU.BOOT0, IC1MCU.VSSA, IC1PWR.VSS@1, IC1PWR.VSS@2, IC2A.G, IC2B.G, IC2P.GND, IC3A.G, IC3B.G, IC3P.GND, IC4.GND, IC5.GND, JP1.GND, JP2.4, JP4.9, JP5.3, R3.1, R7.2; no longer C1.1, C19.-, C2.1, C21.2, C22.2, C23.2, C24.-, C25.2, C4.-, C6.2, C7.2, IC1A.G, IC1B.G, IC1P.GND, IC2.GND, IC3.GND, IC4MCU.BOOT0, IC4MCU.VSSA, IC4PWR.VSS@1, IC4PWR.VSS@2, IC5A.G, IC5B.G, IC5P.GND, J3.GND, JP1.4, JP2.3, R2.1
- net LAT: now also IC1MCU.PB5, IC2B.A1; no longer IC4MCU.PB5, IC5B.A1
- net LAT_H: now also IC2B.Y1; no longer IC5B.Y1
- net MISO: now also IC5.GPIO12, JP1.DATA0/MISO; no longer IC2.GPIO12, J3.DATA0/MISO
- net MOSI: now also IC5.GPIO4, JP1.CMD/MOSI; no longer IC2.GPIO4, J3.CMD/MOSI
- net N$1: now also R4.1, S1.S, S1.S1; no longer R5.1, S2.S, S2.S1
- net N$2: now also IC1MCU.VCAP1; no longer IC4MCU.VCAP1
- net N$3: now also C6.+, IC1MCU.VCAP2; no longer C4.+, IC4MCU.VCAP2
- net OE: now also IC1MCU.PB6, IC3B.A4; no longer IC1B.A4, IC4MCU.PB6
- net OE_H: now also IC3B.Y4; no longer IC1B.Y4
- net R0: now also IC1MCU.PC0, IC3A.A1; no longer IC1A.A1, IC4MCU.PC0
- net R0_H: now also IC3A.Y1; no longer IC1A.Y1
- net R1: now also IC1MCU.PC3, IC3A.A3; no longer IC1A.A3, IC4MCU.PC3
- net R1_H: now also IC3A.Y3; no longer IC1A.Y3
- net RESET: now also C13.1, IC1MCU.NRST, IC5.REST, JP5.5, R5.1, S2.S, S2.S1; no longer C22.1, IC2.REST, IC4MCU.NRST, JP2.5, R1.1, S1.S, S1.S1
- net RX: now also IC1MCU.PA3, IC5.GPIO15, R3.2; no longer IC2.GPIO15, IC4MCU.PA3, R2.2
- net SCLK: now also IC5.GPIO14, JP1.CLK; no longer IC2.GPIO14, J3.CLK
- net SDCS: now also IC5.GPIO5, JP1.DATA3-CD/CS_N; no longer IC2.GPIO5, J3.DATA3-CD/CS_N
- net SWCLK: now also IC1MCU.PA14, JP5.2; no longer IC4MCU.PA14, JP2.2
- net SWDIO: now also IC1MCU.PA13, JP5.4; no longer IC4MCU.PA13, JP2.4
- net TX: now also IC1MCU.PA2, IC5.GPIO13; no longer IC2.GPIO13, IC4MCU.PA2
Other:
- note added: "EXTERNAL BUTTONS"
- note added: "Reserved for extra display signals"
- note added: "STM32 and ESP8266"
- note removed: "STM32 and ESP8266 wiring."

Commit message: board rev b final final
Parts:
- IC5: value (none) -> ESP8266-12E/ESP-12E; device esp12e:ESP8266-12EESP12E -> ESP8266-12E_ESP-12E:ESP8266-12E/ESP-12E
Connections:
- net +3V3: now also IC5.EN; no longer IC5.CH_PD
- net DEBUG_TX: now also IC5.IO2; no longer IC5.GPIO2
- net FLASH: now also IC5.IO0; no longer IC5.GPIO0
- net MISO: now also IC5.IO12; no longer IC5.GPIO12
- net MOSI: now also IC5.IO4; no longer IC5.GPIO4
- net RESET: now also IC5.RESET; no longer IC5.REST
- net RX: now also IC5.IO15; no longer IC5.GPIO15
- net SCLK: now also IC5.IO14; no longer IC5.GPIO14
- net SDCS: now also IC5.IO5; no longer IC5.GPIO5
- net TX: now also IC5.IO13; no longer IC5.GPIO13
Other:
- moved on the sheet: C1, C2, IC5, R1, R2, R3
