File: board/contbrd.brd (EAGLE design)
At the start: 97.8 x 65.8 mm, 33 parts, among them IC1 74HCT244DW, IC3 LM3940, IC4 STM32F205RGT, IC5 74HCT244DW, J1 DCJ0202, J3 DM3AT-SF-PEJM5

Commit message: mb
Routing:
- net +5V: track 117.7 -> 110.9 mm
- net RESET: track 121.7 -> 123.9 mm
- net G0_H: track 32.0 -> 31.2 mm
- net ESP_PROG_TX: track 22.9 -> 23.5 mm
- net OE_H: track 38.6 -> 38.0 mm
- net R0: track 32.8 -> 32.2 mm
- net C_H: track 31.7 -> 32.2 mm
- net A_H: track 30.2 -> 30.7 mm
- added copper zone on layer 16, net +5V
- removed copper zone on layer 1, net +5V

Commit message: board rev b
Parts:
- removed C19: 100uF, rcl:E2,5-6
- removed C21, C25: 100nF, rcl:C025-025X050
- removed J3: DM3AT-SF-PEJM5, connector:DM3AT-SF-PEJM5
- added C11, C12, C14: 100nF, rcl:C025-025X050
- added JP4: (no value), pinhead:1X09
- added JP5: (no value), pinhead:1X06
- added R7: 12k, rcl:0204/7
- C2: value 1uF -> 100uF; device rcl:C050-024X044 -> rcl:E2,5-6
- C3: value 100nF -> 1uF; device rcl:C025-025X050 -> rcl:C050-024X044
- C4: value 2.2uF -> 100nF; device rcl:E1,8-4 -> rcl:C025-025X050
- C6: value 100nF -> 2.2uF; device rcl:C025-025X050 -> rcl:E1,8-4
- IC1: value 74HCT244DW -> STM32F205RGT; device 74xx-eu:SO20W -> micro-stm_v3:LQFP64
- IC2: value (none) -> 74HCT244DW; device esp12e:ESP8266-ESP12E -> 74xx-eu:SO20W
- IC3: value LM3940 -> 74HCT244DW; device LM3940:TO220 -> 74xx-eu:SO20W
- IC4: value STM32F205RGT -> LM3940; device micro-stm_v3:LQFP64 -> LM3940:TO220
- IC5: value 74HCT244DW -> (none); device 74xx-eu:SO20W -> esp12e:ESP8266-ESP12E
- JP1: value (none) -> DM3AT-SF-PEJM5; device pinhead:1X05 -> connector:DM3AT-SF-PEJM5
- JP2: device con-lstb:MA06-1 -> pinhead:1X05
- R4: value 12k -> 470
- R5: value 470 -> 12k
- moved R1 83.3 mm to (95.1, 30.9), turned to 90 degrees
- moved JP2 59.3 mm to (80.0, 55.9), turned to 0 degrees
- moved R5 51.1 mm to (14.6, 52.4), turned to 270 degrees
- moved S1 45.1 mm to (52.6, 58.3)
- moved S2 45.1 mm to (7.62, 54.6)
- moved R4 41.0 mm to (65.2, 59.6), turned to 0 degrees
- moved IC4 40.2 mm to (7.62, 34.3)
- moved JP1 36.2 mm to (78.4, 19.7)
- moved IC2 31.2 mm to (50.8, 22.9)
- moved IC5 31.2 mm to (78.7, 36.8)
- moved C1 28.8 mm to (67.9, 27.4), turned to 270 degrees
- moved IC3 27.6 mm to (32.7, 22.9)
- moved IC1 26.1 mm to (46.4, 45.1)
- moved C2 23.7 mm to (63.3, 27.1), turned to 270 degrees
- moved C7 20.2 mm to (40.3, 30.4), turned to 0 degrees
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- renumbered C20 to C9, C22 to C13, C23 to C8, C24 to C10, J5 to JP3
Connections:
- removed net N$4: C1.2, C2.2, C3.2, IC4.1, IC4.13
- new net ACTLED: IC1.21, JP4.3
- new net MENBTN: IC1.23, JP4.4
- new net NXTBTN: IC1.43, JP4.6
- new net PRVBTN: IC1.42, JP4.5
- new net PWRBTN: IC1.14, JP4.8, R7.1
- new net SELBTN: IC1.41, JP4.7
- new net UPDLED: IC1.22, JP4.2
- net +3V3: now also C1.1, C11.1, C12.1, C14.1, C2.+, C3.2, C4.2, C7.2, IC1.1, IC1.13, IC1.19, IC1.32, IC1.48, IC1.64, IC4.3, IC5.3, IC5.8, JP1.4, JP4.1, JP5.1, R1.1, R2.1, R5.2; no longer C19.+, C21.1, C25.1, C6.1, C7.1, IC2.3, IC2.8, IC3.3, IC4.19, IC4.32, IC4.48, IC4.64, J3.4, JP1.1, R1.2, R3.1, R4.1
- net +5V: now also IC2.20, IC3.20, IC4.1; no longer IC1.20, IC3.1, IC5.20
- net A: now also IC1.26, IC3.11; no longer IC1.11, IC4.26
- net A_H: now also IC3.9; no longer IC1.9
- net B: now also IC1.27, IC2.6; no longer IC4.27, IC5.6
- net B0: now also IC1.10, IC3.4; no longer IC1.4, IC4.10
- net B0_H: now also IC3.16; no longer IC1.16
- net B1: now also IC1.25, IC3.8; no longer IC1.8, IC4.25
- net B1_H: now also IC3.12; no longer IC1.12
- net B_H: now also IC2.14; no longer IC5.14
- net C: now also IC1.28, IC3.13; no longer IC1.13, IC4.28
- net C_H: now also IC3.7; no longer IC1.7
- net D: now also IC1.55, IC2.8; no longer IC4.55, IC5.8
- net DCLK: now also IC1.37, IC3.15; no longer IC1.15, IC4.37
- net DCLK_H: now also IC3.5; no longer IC1.5
- net DEBUG_TX: now also IC5.11, JP2.5, R2.2; no longer IC2.11, JP1.5, R4.2
- net D_H: now also IC2.12; no longer IC5.12
- net ESP_PROG_RX: now also IC5.15, JP2.3; no longer IC2.15, JP1.3
- net ESP_PROG_TX: now also IC5.16, JP2.2; no longer IC2.16, JP1.2
- net FLASH: now also IC5.12, R1.2, R4.2; no longer IC2.12, R3.2, R5.2
- net G0: now also IC1.9, IC2.2; no longer IC4.9, IC5.2
- net G0_H: now also IC2.18; no longer IC5.18
- net G1: now also IC1.24, IC2.4; no longer IC4.24, IC5.4
- net G1_H: now also IC2.16; no longer IC5.16
- net GND: now also C1.2, C11.2, C12.2, C14.2, C2.-, C4.1, C6.-, C7.1, IC1.12, IC1.18, IC1.60, IC1.63, IC2.1, IC2.10, IC2.19, IC3.1, IC3.10, IC3.19, IC4.2, IC5.9, JP1.6, JP1.MOUNT0, JP1.MOUNT1, JP1.MOUNT2, JP1.MOUNT3, JP2.4, JP4.9, JP5.3, R3.1, R7.2; no longer C1.1, C19.-, C2.1, C21.2, C25.2, C4.-, C6.2, C7.2, IC1.1, IC1.10, IC1.19, IC2.9, IC3.2, IC4.12, IC4.18, IC4.60, IC4.63, IC5.1, IC5.10, IC5.19, J3.6, J3.MOUNT0, J3.MOUNT1, J3.MOUNT2, J3.MOUNT3, JP1.4, JP2.3, R2.1
- net LAT: now also IC1.57, IC2.11; no longer IC4.57, IC5.11
- net LAT_H: now also IC2.9; no longer IC5.9
- net MISO: now also IC5.6, JP1.7; no longer IC2.6, J3.7
- net MOSI: now also IC5.13, JP1.3; no longer IC2.13, J3.3
- net N$1: now also R4.1, S1.1, S1.2; no longer R5.1, S2.1, S2.2
- net N$2: now also IC1.31; no longer IC4.31
- net N$3: now also C6.+, IC1.47; no longer C4.+, IC4.47
- net OE: now also IC1.58, IC3.17; no longer IC1.17, IC4.58
- net OE_H: now also IC3.3; no longer IC1.3
- net R0: now also IC1.8, IC3.2; no longer IC1.2, IC4.8
- net R0_H: now also IC3.18; no longer IC1.18
- net R1: now also IC1.11, IC3.6; no longer IC1.6, IC4.11
- net R1_H: now also IC3.14; no longer IC1.14
- net RESET: now also IC1.7, IC5.1, JP5.5, R5.1, S2.1, S2.2; no longer IC2.1, IC4.7, JP2.5, R1.1, S1.1, S1.2
- net RX: now also IC1.17, IC5.10, R3.2; no longer IC2.10, IC4.17, R2.2
- net SCLK: now also IC5.5, JP1.5; no longer IC2.5, J3.5
- net SDCS: now also IC5.14, JP1.2; no longer IC2.14, J3.2
- net SWCLK: now also IC1.49, JP5.2; no longer IC4.49, JP2.2
- net SWDIO: now also IC1.46, JP5.4; no longer IC4.46, JP2.4
- net TX: now also IC1.16, IC5.7; no longer IC2.7, IC4.16
Routing:
- net PRVBTN: track 0.00 -> 70.3 mm, vias 0 -> 1
- net SELBTN: track 0.00 -> 59.3 mm, vias 0 -> 1
- net NXTBTN: track 0.00 -> 58.5 mm, vias 0 -> 1
- net MENBTN: track 0.00 -> 50.0 mm, vias 0 -> 1
- net UPDLED: track 0.00 -> 43.3 mm, vias 0 -> 1
- net PWRBTN: track 0.00 -> 43.3 mm
- net ACTLED: track 0.00 -> 36.4 mm, vias 0 -> 1
- net +3V3: track 32.3 -> 60.6 mm, vias 3 -> 5
- net N$4: track 19.4 -> 0.00 mm
- net GND: track 57.2 -> 59.7 mm, vias 6 -> 7
- net MOSI: track 24.1 -> 22.2 mm
- net SCLK: track 16.4 -> 17.6 mm
- net MISO: track 13.5 -> 14.7 mm
- net B1: track 40.1 -> 40.9 mm
Other:
- board size 97.8 x 65.8 mm -> 97.8 x 66.1 mm
- board text added: "EXT BUTTON"

Commit message: board rev b final final
Parts:
- IC5: value (none) -> ESP8266-12E/ESP-12E; device esp12e:ESP8266-ESP12E -> ESP8266-12E_ESP-12E:XCVR_ESP8266-12E/ESP-12E
- moved R3 5.77 mm to (95.2, 30.9)
- moved C14 3.17 mm to (92.4, 17.3)
- moved R1 2.87 mm to (92.8, 29.2)
- moved R2 2.81 mm to (90.2, 28.0)
- moved JP1 1.93 mm to (80.3, 19.4)
- moved IC5 1.62 mm to (79.1, 35.2)
- moved C2 0.14 mm to (63.4, 27.2)
Connections:
- net DEBUG_TX: now also IC5.17; no longer IC5.11
- net ESP_PROG_RX: now also IC5.21; no longer IC5.15
- net ESP_PROG_TX: now also IC5.22; no longer IC5.16
- net FLASH: now also IC5.18; no longer IC5.12
- net GND: now also IC5.15; no longer IC5.9
- net MOSI: now also IC5.19; no longer IC5.13
- net RX: now also IC5.16; no longer IC5.10
- net SDCS: now also IC5.20; no longer IC5.14
Routing:
- net GND: track 59.7 -> 68.8 mm
- net RX: track 43.0 -> 51.0 mm
- net +3V3: track 60.6 -> 63.9 mm
- net DEBUG_TX: track 34.0 -> 32.4 mm
- net MOSI: track 22.2 -> 20.8 mm
- net SDCS: track 23.7 -> 22.4 mm
- net ESP_PROG_TX: track 23.5 -> 24.5 mm
- net ESP_PROG_RX: track 23.3 -> 24.2 mm
- net D: track 38.8 -> 39.7 mm
- net SCLK: track 17.6 -> 18.4 mm
- net TX: track 24.6 -> 25.2 mm
- net RESET: track 123.9 -> 124.6 mm
Other:
- board text added: "1.6mm thick"
- board text added: "Mounting holes M2"
- board text added: "White soldermask PCB"

Commit message: finish board
Parts:
- moved C14 1.00 mm to (92.1, 16.3)
Routing:
- net G0_H: track 31.2 -> 28.7 mm
- net G1_H: track 27.6 -> 28.9 mm
- net DCLK_H: track 35.8 -> 34.6 mm
- net +3V3: track 63.9 -> 63.1 mm
- net A_H: track 30.7 -> 30.1 mm

Commit message: spacing on brd
Parts:
- moved JP1 1.59 mm to (80.3, 17.8)
Routing:
- net SCLK: track 18.4 -> 20.0 mm
- net SDCS: track 22.4 -> 24.0 mm
- net MOSI: track 20.8 -> 22.4 mm
- net MISO: track 15.2 -> 16.8 mm
- net +3V3: track 63.1 -> 64.4 mm
Changed lines of the file:
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@@
 <drawing>
 <settings>
-<setting alwaysvectorfont="no"/>
+<setting alwaysvectorfont="yes"/>
 <setting verticaltext="up"/>
 </settings>
@@
 <attribute name="VALUE" x="63.5254" y="59.0804" size="0.9906" layer="27" ratio="10"/>
 </element>
-<element name="JP1" library="connector" package="DM3AT-SF-PEJM5" value="DM3AT-SF-PEJM5" x="80.264" y="19.3675" smashed="yes">
-<attribute name="DESCRIPTION" value="CONN MICRO SD CARD PUSH-PUSH R/A" x="80.264" y="19.3675" size="1.27" layer="27" display="off"/>
-<attribute name="DIGIKEY" value="HR1964CT-ND" x="80.264" y="19.3675" size="1.27" layer="27" display="off"/>
-<attribute name="MANUFACTURER" value="Hirose Electric Co Ltd" x="80.264" y="19.3675" size="1.27" layer="27" display="off"/>
-<attribute name="MPN" value="DM3AT-SF-PEJM5" x="80.264" y="19.3675" size="1.27" layer="27" display="off"/>
-<attribute name="NAME" x="73.0825" y="19.877" size="1.016" layer="25" ratio="12" align="bottom-center"/>
+<element name="JP1" library="connector" package="DM3AT-SF-PEJM5" value="DM3AT-SF-PEJM5" x="80.264" y="17.78" smashed="yes">
+<attribute name="DESCRIPTION" value="CONN MICRO SD CARD PUSH-PUSH R/A" x="80.264" y="17.78" size="1.27" layer="27" display="off"/>
+<attribute name="DIGIKEY" value="HR1964CT-ND" x="80.264" y="17.78" size="1.27" layer="27" display="off"/>
+<attribute name="MANUFACTURER" value="Hirose Electric Co Ltd" x="80.264" y="17.78" size="1.27" layer="27" display="off"/>
+<attribute name="MPN" value="DM3AT-SF-PEJM5" x="80.264" y="17.78" size="1.27" layer="27" display="off"/>
+<attribute name="NAME" x="73.0825" y="18.2895" size="1.016" layer="25" ratio="12" align="bottom-center"/>
 </element>
 <element name="J2" library="SparkFun-Connectors" package="SCREWTERMINAL-5MM-2" value="" x="21.971" y="6.35" smashed="yes">
@@
 <wire x1="42.545" y1="51.435" x2="42.605" y2="51.375" width="0.1524" layer="1"/>
 <wire x1="42.605" y1="51.375" x2="42.605" y2="50.835" width="0.1524" layer="1"/>
-<wire x1="92.075" y1="17.5895" x2="81.153" y2="17.5895" width="0.254" layer="1"/>
-<wire x1="81.153" y1="17.5895" x2="80.164" y2="18.5785" width="0.254" layer="1"/>
-<wire x1="80.164" y1="18.5785" x2="80.164" y2="19.2675" width="0.254" layer="1"/>
+<wire x1="92.075" y1="17.5895" x2="90.17" y2="15.6845" width="0.254" layer="1"/>
+<wire x1="90.17" y1="15.6845" x2="80.8355" y2="15.6845" width="0.254" layer="1"/>
+<wire x1="80.164" y1="17.68" x2="80.164" y2="16.356" width="0.254" layer="1"/>
+<wire x1="80.8355" y1="15.6845" x2="80.164" y2="16.356" width="0.254" layer="1"/>
 <contactref element="JP4" pad="1"/>
 <via x="66.04" y="44.7675" extent="1-16" drill="0.35"/>
@@
 <signal name="SCLK">
 <contactref element="JP1" pad="5"/>
-<wire x1="79.064" y1="19.2675" x2="79.064" y2="19.8977125" width="0.1524" layer="1"/>
+<wire x1="79.064" y1="17.68" x2="79.064" y2="19.8977125" width="0.1524" layer="1"/>
 <wire x1="79.064" y1="19.8977125" x2="74.9739" y2="23.9878125" width="0.1524" layer="1"/>
 <wire x1="74.9739" y1="23.9878125" x2="74.9739" y2="28.2136" width="0.1524" layer="1"/>
@@
 <via x="81.28" y="22.5425" extent="1-16" drill="0.35"/>
 <wire x1="81.28" y1="22.5425" x2="81.264" y2="22.5265" width="0.1524" layer="1"/>
-<wire x1="81.264" y1="22.5265" x2="81.264" y2="19.2675" width="0.1524" layer="1"/>
+<wire x1="81.264" y1="22.5265" x2="81.264" y2="17.68" width="0.1524" layer="1"/>
 <wire x1="84.455" y1="36.5125" x2="84.455" y2="25.7175" width="0.1524" layer="16"/>
 <wire x1="84.455" y1="25.7175" x2="81.28" y2="22.5425" width="0.1524" layer="16"/>
@@
 <signal name="MISO">
 <contactref element="JP1" pad="7"/>
-<wire x1="76.864" y1="19.2675" x2="76.864" y2="19.7582875" width="0.1524" layer="1"/>
+<wire x1="76.864" y1="17.68" x2="76.864" y2="19.7582875" width="0.1524" layer="1"/>
 <wire x1="76.864" y1="19.7582875" x2="73.025" y2="23.5972875" width="0.1524" layer="1"/>
 <contactref element="IC5" pad="6"/>
@@
 <via x="82.423" y="24.892" extent="1-16" drill="0.35"/>
 <wire x1="82.423" y1="24.892" x2="82.364" y2="24.833" width="0.1524" layer="1"/>
-<wire x1="82.364" y1="24.833" x2="82.364" y2="19.2675" width="0.1524" layer="1"/>
+<wire x1="82.364" y1="24.833" x2="82.364" y2="17.68" width="0.1524" layer="1"/>
 <wire x1="83.8482" y1="26.3172" x2="83.8482" y2="38.1282" width="0.1524" layer="16"/>
 <wire x1="83.8482" y1="38.1282" x2="84.1375" y2="38.4175" width="0.1524" layer="16"/>
