File: board/rev2/matrixandbuffer.kicad_sch (KiCad schematic)
At the start: 0 parts

Commit message: Finish most of power section of rev2 PCB
Parts:
- added J4: Conn_02x08_Odd_Even, Connector_IDC:IDC-Header_2x08_P2.54mm_Vertical, symbol Connector_Generic:Conn_02x08_Odd_Even
- added U2, U9: 74AHCT244, symbol 74xx:74AHCT244
Connections:
- new net +5V: U2.20 (VCC), U9.20 (VCC)
- new net GND: U2.10 (GND), U9.10 (GND)

Commit message: More board stuff
(better clk routing, etc.)
Parts:
- removed J4: Conn_02x08_Odd_Even, Connector_IDC:IDC-Header_2x08_P2.54mm_Vertical, symbol Connector_Generic:Conn_02x08_Odd_Even
- removed U2, U9: 74AHCT244, symbol 74xx:74AHCT244
- added J4: Conn_02x08_Counter_Clockwise, symbol Connector_Generic:Conn_02x08_Counter_Clockwise
- added U12: 74HC245, symbol 74xx:74HC245
